Commit message: output map to txt get map>bfp transform

File: src/config/tb3_description.urdf (robot description, URDF)
Before this commit: robot turtlebot3_burger, 6 links, 5 joints
Links:
- added link imu_link, mass mass; collision box size=0.1 0.1 0.1; visual box size=0.1 0.1 0.1
Joints:
- added joint imu_joint: type fixed, parent base_link, child imu_link, origin xyz=-0.032 0 0.172 rpy=0 0 0
- joint lidar_joint: origin xyz=0 0 0.0 rpy=0 0 0 -> xyz=-0.032 0 0.172 rpy=0 0 0

File: src/config/tb_descript_temp.urdf (robot description, URDF)
Before this commit: robot turtlebot3_burger, 4 links, 3 joints
Links:
- added link imu_link; collision box size=0.1 0.1 0.1; visual box size=0.1 0.1 0.1
Joints:
- added joint imu_joint: type fixed, parent base_link, child imu_link, origin xyz=-0.032 0 0.172 rpy=0 0 0
- joint lidar_joint: origin xyz=0 0 0.0 rpy=0 0 0 -> xyz=-0.032 0 0.172 rpy=0 0 0
